Commit message: Driving robot simulation

File: description/robot_core.xacro (robot description, xacro)
@@ -37,8 +37,11 @@
             </geometry>
         </collision>
-        <xacro:inertial_box mass="0.5" x="0.2286" y="0.097" z="0.1">
-            <origin xyz ="0.1143 0 0.05" rpy="0 0 0"/>
+        <xacro:inertial_box mass="2" x="0.2286" y="0.097" z="0.1">
+            <origin xyz ="0.1143 0 0.5" rpy="0 0 0"/>
         </xacro:inertial_box>
     </link>
+    <gazebo reference="chassis">
+        <material>Gazebo/White</material>
+    </gazebo>
     <!--LEFT BACK WHEEL LINK -->
     <joint name="left_back_wheel_joint" type="continuous">
@@ -64,4 +67,7 @@
         </xacro:inertial_cylinder>
     </link>
+    <gazebo reference="left_back_wheel">
+        <material>Gazebo/Blue</material>
+    </gazebo>
     <!--RIGHT BACK WHEEL LINK -->
     <joint name="right_back_wheel_joint" type="continuous">
@@ -87,49 +93,32 @@
         </xacro:inertial_cylinder>
     </link>
-    <!--LEFT FRONT WHEEL LINK -->
-    <joint name="left_front_wheel_joint" type="continuous">
+    <gazebo reference="right_back_wheel">
+        <material>Gazebo/Blue</material>
+    </gazebo>
+    <joint name="caster_wheel_joint" type="fixed">
         <parent link="base_link"/>
-        <child link="left_front_wheel" />
-        <origin xyz="0.0381 0.061 0" rpy="-${pi/2} 0 0" />
-        <axis xyz="0 0 1" />
+        <child link="caster_wheel"/>
+        <origin xyz="0.07 0 0"/>
     </joint>
-    <link name="left_front_wheel">
+    <link name="caster_wheel">
         <visual>
             <geometry>
-                <cylinder radius="0.03175" length="0.025" />
+                <sphere radius="0.03175"/>
             </geometry>
-            <material name="blue" />
+            <material nasme="black"/>
         </visual>
         <collision>
             <geometry>
-                <cylinder radius="0.03175" length="0.025" />
+                <sphere radius="0.03175"/>
             </geometry>
         </collision>
-        <xacro:inertial_cylinder mass="0.1" radius="0.03175" length="0.025">
-            <origin xyz ="0 0 0" rpy="0 0 0"/>
-        </xacro:inertial_cylinder>
+        <xacro:inertial_sphere mass="0.1" radius="0.03175">
+            <origin xyz="0 0 0" rpy="0 0 0"/>
+        </xacro:inertial_sphere>
     </link>
-    <!--RIGHT FRONT WHEEL LINK -->
-    <joint name="right_front_wheel_joint" type="continuous">
-            <parent link="base_link"/>
-            <child link="right_front_wheel" />
-            <origin xyz="0.0381 -0.061 0" rpy="${pi/2} 0 0" />
-            <axis xyz="0 0 -1" />
-    </joint>
-    <link name="right_front_wheel">
-        <visual>
-            <geometry>
-                <cylinder radius="0.03175" length="0.025" />
-            </geometry>
-            <material name="blue" />
-        </visual>
-        <collision>
-            <geometry>
-                <cylinder radius="0.03175" length="0.025" />
-            </geometry>
-        </collision>
-        <xacro:inertial_cylinder mass="0.1" radius="0.03175" length="0.025">
-            <origin xyz ="0 0 0" rpy="0 0 0"/>
-        </xacro:inertial_cylinder>
-    </link>
+    <gazebo reference="caster_wheel">
+        <material>Gazebo/Black</material>
+        <mu1 value="0.0001"/>
+        <mu2 value="0.0001"/>
+    </gazebo>
 </robot>

Commit message: Updated Core to Tuttorial

File: description/robot_core.xacro (robot description, xacro)
@@ -21,22 +21,22 @@
         <parent link="base_link" />
         <child link="chassis" />
-        <origin xyz="-0.1143 0 0" />
+        <origin xyz="-0.1 0 0"/>
     </joint>
     <link name="chassis">
         <visual>
-            <origin xyz="0.1143 0 0.05" />
-            <geometry>
-                <box size="0.2286 0.097 0.1" />
-            </geometry>
-            <material name="white" />
-        </visual>
+        <origin xyz="0.15 0 0.075" rpy="0 0 0"/>
+        <geometry>
+            <box size="0.3 0.3 0.15"/>
+        </geometry>
+        <material name="white"/>
+    </visual>
         <collision>
-            <origin xyz="0.1143 0 0.05" />
-            <geometry>
-                <box size="0.2286 0.097 0.1" />
-            </geometry>
+            <origin xyz="0.15 0 0.075" rpy="0 0 0"/>
+        <geometry>
+            <box size="0.3 0.3 0.15"/>
+        </geometry>
         </collision>
-        <xacro:inertial_box mass="2" x="0.2286" y="0.097" z="0.1">
-            <origin xyz ="0.1143 0 0.5" rpy="0 0 0"/>
+        <xacro:inertial_box mass="0.5" x="0.3" y="0.3" z="0.15">
+            <origin xyz="0.15 0 0.075" rpy="0 0 0"/>
         </xacro:inertial_box>
     </link>
@@ -48,11 +48,11 @@
             <parent link="base_link"/>
             <child link="left_back_wheel" />
-            <origin xyz="-0.0381 0.061 0" rpy="-${pi/2} 0 0" />
-            <axis xyz="0 0 1" />
+            <origin xyz="0 0.175 0" rpy="-${pi/2} 0 0"/>
+            <axis xyz="0 0 1"/>
     </joint>
     <link name="left_back_wheel">
         <visual>
             <geometry>
-                <cylinder radius="0.03175" length="0.025" />
+                <cylinder length="0.04" radius="0.05" />
             </geometry>
             <material name="blue" />
@@ -60,9 +60,9 @@
         <collision>
             <geometry>
-                <cylinder radius="0.03175" length="0.025" />
+                <cylinder length="0.04" radius="0.05" />
             </geometry>
         </collision>
-        <xacro:inertial_cylinder mass="0.1" radius="0.03175" length="0.025">
-            <origin xyz ="0 0 0" rpy="0 0 0"/>
+        <xacro:inertial_cylinder mass="0.1" length="0.05" radius="0.05">
+            <origin xyz="0 0 0" rpy="0 0 0"/>
         </xacro:inertial_cylinder>
     </link>
@@ -74,5 +74,5 @@
             <parent link="base_link"/>
             <child link="right_back_wheel" />
-            <origin xyz="-0.0381 -0.061 0" rpy="${pi/2} 0 0" />
+            <origin xyz="0 -0.175 0" rpy="${pi/2} 0 0"/>
             <axis xyz="0 0 -1" />
     </joint>
@@ -80,5 +80,5 @@
         <visual>
             <geometry>
-                <cylinder radius="0.03175" length="0.025" />
+                <cylinder length="0.04" radius="0.05" />
             </geometry>
             <material name="blue" />
@@ -86,9 +86,9 @@
         <collision>
             <geometry>
-                <cylinder radius="0.03175" length="0.025" />
+                <cylinder length="0.04" radius="0.05" />
             </geometry>
         </collision>
-        <xacro:inertial_cylinder mass="0.1" radius="0.03175" length="0.025">
-            <origin xyz ="0 0 0" rpy="0 0 0"/>
+        <xacro:inertial_cylinder mass="0.1" length="0.05" radius="0.05">
+            <origin xyz="0 0 0" rpy="0 0 0"/>
         </xacro:inertial_cylinder>
     </link>
@@ -96,22 +96,23 @@
         <material>Gazebo/Blue</material>
     </gazebo>
+    <!--CASTER WHEEL -->
     <joint name="caster_wheel_joint" type="fixed">
         <parent link="base_link"/>
         <child link="caster_wheel"/>
-        <origin xyz="0.07 0 0"/>
+        <origin xyz="0.12 0 0" rpy="0 0 0"/>
     </joint>
     <link name="caster_wheel">
         <visual>
             <geometry>
-                <sphere radius="0.03175"/>
+                <sphere radius="0.05" />
             </geometry>
-            <material nasme="black"/>
+            <material name="black"/>
         </visual>
         <collision>
             <geometry>
-                <sphere radius="0.03175"/>
+                <sphere radius="0.05" />
             </geometry>
         </collision>
-        <xacro:inertial_sphere mass="0.1" radius="0.03175">
+        <xacro:inertial_sphere mass="0.1" radius="0.05">
             <origin xyz="0 0 0" rpy="0 0 0"/>
         </xacro:inertial_sphere>
